File: hardware/watchular_hardware_design/esp32c3_boiler_plate.kicad_sch (KiCad schematic)
At the start: 26 parts, among them J1 USB4105-GF-A, U1 ESP32-C3FH4, U2 MIC5524-3.3YMT-TZ, U3 W25Q16JVSSIQ, Y1 40MHz

Commit message: Updated the file naming to the boiler plate.
Other:
- title: Watchular - 4 x 7 seven segment display -> boiler plate for esp32c3
Changed lines of the file:
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@@
   (paper "A4")
   (title_block
-    (title "Watchular - 4 x 7 seven segment display")
+    (title "boiler plate for esp32c3")
     (date "2022-06-17")
     (rev "v0.1")
