File: hardware/watchular_hardware_design/esp32c3_boilerplate.kicad_pcb (KiCad board)
At the start: 2 copper layers, 26 parts, among them J1 USB4105-GF-A, U1 ESP32-C3FH4, U2 MIC5524-3.3YMT-TZ, U3 W25Q16JVSSIQ, Y1 40MHz

Commit message: Added ESD protection on the USB.
Parts:
- added DA1: SR05, ESD_protection-SR05:SOT143, F.Cu at (111.8, 63.5)
- C10: value 1pF -> 10nF; footprint Capacitor_SMD:C_0402_1005Metric -> Inductor_SMD:L_0402_1005Metric
- C7: value 100nF -> 1pF; footprint Inductor_SMD:L_0402_1005Metric -> Capacitor_SMD:C_0402_1005Metric
- C8: value 1uF -> 100nF
- C9: value 10nF -> 1uF
- L1: value 39nH -> 2.7 nH
- L2: value 2.7 nH -> 3.9 nH
- L3: value 3.9 nH -> 39nH
- R3: footprint Resistor_SMD:R_0402_1005Metric -> Resistor_SMD:R_01005_0402Metric_Pad0.57x0.30mm_HandSolder
Connections:
- C1 pad 1: XTAL_N -> XTAL_P
- C10 pad 1: antenna -> +3.3VA
- C10 pad 2: Net-(C10-Pad2) -> GND
- C7 pad 1: +3V3 -> antenna
- C7 pad 2: GND -> Net-(C7-Pad2)
- C8 pad 1: +3.3VA -> +3V3
- L1 pad 1: +3V3 -> GND
- L1 pad 2: +3.3VA -> Net-(C7-Pad2)
- L2 pad 1: GND -> Net-(C7-Pad2)
- L2 pad 2: Net-(C10-Pad2) -> Net-(AE1-Pad1)
- L3 pad 1: Net-(C10-Pad2) -> +3V3
- L3 pad 2: Net-(AE1-Pad1) -> +3.3VA
- R2 pad 2: XTAL_P -> XTAL_N
- Y1 pad 1: XTAL_N -> XTAL_P
