File: hardware/watchular_hardware_design/watchular_hardware_design.kicad_pcb (KiCad board)
At the start: 4 copper layers, 55.5 x 22.9 mm, 89 parts, among them J1 USB4105-GF-A, J2 665102131822, J3 TSW-116-07-H-S, J4 TSW-116-07-H-S, Q1 BSS123, Q2 BSS123, Q3 BSS123, Q4 BSS123, Q5 Q_PMOS_GSD, U1 MCP73832T-2DCI/OT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

Commit message: Added custom graphics.
Parts:
- added G***: LOGO, custom_graphics:heart, B.Cu at (142.8, 124.0)
Other:
- board text added: "Boris"
- board text added: "for my dear Beatrice"
- board text removed: "Lilordag"
Changed lines of the file:
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@@
       (layer "F.SilkS" (type "Top Silk Screen") (color "White"))
       (layer "F.Paste" (type "Top Solder Paste"))
-      (layer "F.Mask" (type "Top Solder Mask") (color "Blue") (thickness 0.01))
+      (layer "F.Mask" (type "Top Solder Mask") (color "Green") (thickness 0.01))
       (layer "F.Cu" (type "copper") (thickness 0.035))
       (layer "dielectric 1" (type "core") (thickness 0.2104) (material "FR4") (epsilon_r 4.5) (loss_tangent 0.02))
@@
       (layer "dielectric 3" (type "core") (thickness 0.2104) (material "FR4") (epsilon_r 4.5) (loss_tangent 0.02))
       (layer "B.Cu" (type "copper") (thickness 0.035))
-      (layer "B.Mask" (type "Bottom Solder Mask") (color "Blue") (thickness 0.01))
+      (layer "B.Mask" (type "Bottom Solder Mask") (color "Green") (thickness 0.01))
       (layer "B.Paste" (type "Bottom Solder Paste"))
       (layer "B.SilkS" (type "Bottom Silk Screen") (color "White"))
@@
     )
   )
+  (footprint "custom_graphics:heart" (layer "B.Cu")
+    (at 142.8 124.025 -90)
+    (attr board_only exclude_from_pos_files exclude_from_bom)
+    (fp_text reference "G***" (at 0 0 90) (layer "B.SilkS") hide
+      (effects (font (size 1.524 1.524) (thickness 0.3)) (justify mirror))
+    )
+    (fp_text value "LOGO" (at 0.75 0 90) (layer "B.SilkS") hide
+      (effects (font (size 1.524 1.524) (thickness 0.3)) (justify mirror))
+    )
+    (fp_poly (pts
+        (xy 1.266063 1.724738)
+        (xy 1.457941 1.666574)
+        (xy 1.600553 1.59305)
+        (xy 1.752843 1.473541)
+        (xy 1.886089 1.324187)
+        (xy 1.99268 1.155574)
+        (xy 2.065 0.978291)
+        (xy 2.077904 0.929268)
+        (xy 2.097706 0.783692)
+        (xy 2.098139 0.616993)
+        (xy 2.079796 0.44754)
+        (xy 2.059173 0.348839)
+        (xy 2.006395 0.183246)
+        (xy 1.931961 0.018384)
+        (xy 1.833804 -0.148009)
+        (xy 1.709858 -0.318198)
+        (xy 1.558058 -0.494446)
+        (xy 1.376337 -0.679017)
+        (xy 1.162629 -0.874175)
+        (xy 0.914869 -1.082183)
+        (xy 0.630989 -1.305306)
+        (xy 0.372705 -1.498998)
+        (xy 0.262063 -1.580196)
+        (xy 0.163974 -1.651581)
+        (xy 0.08382 -1.709285)
+        (xy 0.026987 -1.74944)
+        (xy -0.001143 -1.768177)
+        (xy -0.003126 -1.769061)
+        (xy -0.022514 -1.756278)
+        (xy -0.072166 -1.72111)
+        (xy -0.146721 -1.667425)
+        (xy -0.24082 -1.599087)
+        (xy -0.349103 -1.519964)
+        (xy -0.384041 -1.494342)
+        (xy -0.711467 -1.24772)
+        (xy -0.999845 -1.016572)
+        (xy -1.250772 -0.79888)
+        (xy -1.465848 -0.592622)
+        (xy -1.646668 -0.39578)
+        (xy -1.794833 -0.206334)
+        (xy -1.911938 -0.022264)
+        (xy -1.999582 0.15845)
+        (xy -2.059364 0.337827)
+        (xy -2.09288 0.517888)
+        (xy -2.101917 0.677144)
+        (xy -2.081051 0.890958)
+        (xy -2.020705 1.092183)
+        (xy -1.924254 1.275815)
+        (xy -1.795077 1.436852)
+        (xy -1.636549 1.570291)
+        (xy -1.452047 1.671127)
+        (xy -1.423202 1.682798)
+        (xy -1.245908 1.730563)
+        (xy -1.051096 1.747147)
+        (xy -0.851913 1.733276)
+        (xy -0.661503 1.689673)
+        (xy -0.523003 1.633197)
+        (xy -0.40913 1.558113)
+        (xy -0.293257 1.452485)
+        (xy -0.185705 1.328273)
+        (xy -0.096798 1.197432)
+        (xy -0.036858 1.07192)
+        (xy -0.035785 1.068851)
+        (xy -0.008638 0.990439)
+        (xy 0.063692 1.137362)
+        (xy 0.134823 1.25728)
+        (xy 0.227795 1.379034)
+        (xy 0.331608 1.490193)
+        (xy 0.435263 1.578322)
+        (xy 0.479811 1.607675)
+        (xy 0.660977 1.689636)
+        (xy 0.858477 1.736388)
+        (xy 1.063207 1.748049)
+      ) (layer "B.SilkS") (width 0) (fill solid))
+  )
   (footprint "Resistor_SMD:R_0402_1005Metric_Pad0.72x0.64mm_HandSolder" locked (layer "B.Cu")
     (at 137.5 126)
@@
     (effects (font (size 0.918 0.918) (thickness 0.15)))
   )
-  (gr_text "Lilordag" (at 141.55 113.1) (layer "F.SilkS")
+  (gr_text "Boris" (at 93.15 112.725) (layer "F.SilkS")
+    (effects (font (size 0.918 0.918) (thickness 0.15)))
+  )
+  (gr_text "for my\ndear\nBeatrice" (at 141.55 113.1) (layer "F.SilkS")
     (effects (font (size 0.918 0.918) (thickness 0.15)))
   )
